Commit message: feat: harmonic potential field done.

File: src/phi_turtlebot3_description/urdf/turtlebot3_burger.urdf (robot description, URDF)
Before this commit: robot turtlebot3_burger, 7 links, 6 joints
Links:
- link ${namespace}base_link: geometry collision box size=0.140 0.140 0.143; visual mesh filename=package://phi_turtlebot3_description/meshes/bases/burger_ba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 scale=0.001 0.001 0.001
- link ${namespace}base_scan: geometry collision cylinder length=0.0315 radius=0.055; visual mesh filename=package://phi_turtlebot3_description/meshes/sensors/lds.stl scale=0.001 0.001 0.001
- link ${namespace}wheel_left_link: geometry collision cylinder length=0.018 radius=0.033; visual mesh filename=package://phi_turtlebot3_description/meshes/wheels/left_tir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 scale=0.001 0.001 0.001
- link ${namespace}wheel_right_link: geometry collision cylinder length=0.018 radius=0.033; visual mesh filename=package://phi_turtlebot3_description/meshes/wheels/right_ti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 scale=0.001 0.001 0.001

File: src/phi_turtlebot3_description/urdf/turtlebot3_burger_cam.urdf (robot description, URDF)
Before this commit: robot turtlebot3_burger_cam, 9 links, 8 joints
Links:
- link ${namespace}base_link: geometry collision box size=0.140 0.140 0.143; visual mesh filename=package://phi_turtlebot3_description/meshes/bases/burger_ba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 scale=0.001 0.001 0.001
- link ${namespace}base_scan: geometry collision cylinder length=0.0315 radius=0.055; visual mesh filename=package://phi_turtlebot3_description/meshes/sensors/lds.stl scale=0.001 0.001 0.001
- link ${namespace}wheel_left_link: geometry collision cylinder length=0.018 radius=0.033; visual mesh filename=package://phi_turtlebot3_description/meshes/wheels/left_tir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 scale=0.001 0.001 0.001
- link ${namespace}wheel_right_link: geometry collision cylinder length=0.018 radius=0.033; visual mesh filename=package://phi_turtlebot3_description/meshes/wheels/right_ti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 scale=0.001 0.001 0.001

File: src/phi_turtlebot3_description/urdf/turtlebot3_waffle.urdf (robot description, URDF)
Before this commit: robot turtlebot3_waffle, 13 links, 12 joints
Links:
- link ${namespace}base_link: geometry collision box size=0.266 0.266 0.094; visual mesh filename=package://phi_turtlebot3_description/meshes/bases/waffle_ba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 scale=0.001 0.001 0.001
- link ${namespace}base_scan: geometry collision cylinder length=0.0315 radius=0.055; visual mesh filename=package://phi_turtlebot3_description/meshes/sensors/lds.stl scale=0.001 0.001 0.001
- link ${namespace}camera_link: geometry collision box size=0.012 0.132 0.020; visual mesh filename=package://phi_turtlebot3_description/meshes/sensors/r200.dae
- link ${namespace}wheel_left_link: geometry collision cylinder length=0.018 radius=0.033; visual mesh filename=package://phi_turtlebot3_description/meshes/wheels/left_tir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 scale=0.001 0.001 0.001
- link ${namespace}wheel_right_link: geometry collision cylinder length=0.018 radius=0.033; visual mesh filename=package://phi_turtlebot3_description/meshes/wheels/right_ti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 scale=0.001 0.001 0.001

File: src/phi_turtlebot3_description/urdf/turtlebot3_waffle_pi.urdf (robot description, URDF)
Before this commit: robot turtlebot3_waffle_pi, 11 links, 10 joints
Links:
- link ${namespace}base_link: geometry collision box size=0.266 0.266 0.094; visual mesh filename=package://phi_turtlebot3_description/meshes/bases/waffle_pi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 scale=0.001 0.001 0.001
- link ${namespace}base_scan: geometry collision cylinder length=0.0315 radius=0.055; visual mesh filename=package://phi_turtlebot3_description/meshes/sensors/lds.stl scale=0.001 0.001 0.001
- link ${namespace}wheel_left_link: geometry collision cylinder length=0.018 radius=0.033; visual mesh filename=package://phi_turtlebot3_description/meshes/wheels/left_tir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 scale=0.001 0.001 0.001
- link ${namespace}wheel_right_link: geometry collision cylinder length=0.018 radius=0.033; visual mesh filename=package://phi_turtlebot3_description/meshes/wheels/right_ti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 scale=0.001 0.001 0.001
